File: BuckConverter/BuckConverter.kicad_sch (KiCad schematic)
At the start: 0 parts

Commit message: andrew testing respirtory
Other:
- note added: "TESTING KICAD + GITHUB (Andrew Nguyen)"
Changed lines of the file:
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@@
 		(rev "v0")
+	)
+	(text "TESTING KICAD + GITHUB (Andrew Nguyen)"
+		(exclude_from_sim no)
+		(at 70.104 119.888 0)
+		(effects
+			(font
+				(size 1.27 1.27)
+			)
+		)
 	)
 	(label "PWM"
